Commit message: Fix camera and add hull

File: urdf/izzyboat.urdf (robot description, URDF)
Before this commit: robot izzyboat, 2 links, 1 joints
Links:
- added link izzy/camera_forward_optical; visual box size=.5 .3 .01
- link izzy/base_link: geometry visual box size=0.55 0.55 0.3; visual box size=1.3 0.8 0.3
Joints:
- added joint camera_forward_to_camera_forward_optical: type fixed, parent izzy/camera_forward, child izzy/camera_forward_optical, origin xyz=0 0 0 rpy=-1.57075 0 -1.57075
- joint base_to_camera_forward: origin xyz=1.8 0 -0.055 -> xyz=1.8 0 -0.055 rpy=0 0 0

Commit message: Update for cuav gps ref point

File: urdf/izzyboat.urdf (robot description, URDF)
Before this commit: robot izzyboat, 3 links, 2 joints
Links:
- added link base_link
Joints:
- added joint base_to_izzy: type fixed, parent base_link, child izzy/base_link, origin xyz=0 0 0 rpy=0 0 0
- joint base_to_camera_forward: origin xyz=1.8 0 -0.055 rpy=0 0 0 -> xyz=1.55 0 -0.055 rpy=0 0 0

Commit message: Disable unused usb camera launch nodes

File: urdf/izzyboat.urdf (robot description, URDF)
Before this commit: robot izzyboat, 4 links, 3 joints
Links:
- removed link base_link
- added link izzy/sensors/cameras/oak_rgb_camera_optical_frame
Joints:
- removed joint base_to_izzy
- added joint forward_optical_to_oak_optical: type fixed, parent izzy/camera_forward_optical, child izzy/sensors/cameras/oak_rgb_camera_optical_frame, origin xyz=0 0 0 rpy=0 0 0

Commit message: Add deltat frame

File: urdf/izzyboat.urdf (robot description, URDF)
Before this commit: robot izzyboat, 4 links, 3 joints
Links:
- added link izzy/deltat
Joints:
- added joint base_to_deltat: type fixed, parent izzy/base_link, child izzy/deltat, origin xyz=0 0 0 rpy=3.14159 0 0

Commit message: Use tf for static transforms, not tf_static

File: urdf/izzyboat.urdf (robot description, URDF)
Before this commit: robot izzyboat, 5 links, 4 joints
Links:
- link izzy/deltat: geometry visual box size=0.1 0.1 0.1
Joints:
- joint base_to_deltat: origin xyz=0 0 0 rpy=3.14159 0 0 -> xyz=0 0 -0.65 rpy=3.14159 0 0

Commit message: Add DeltaT

File: urdf/izzyboat.urdf (robot description, URDF)
Before this commit: robot izzyboat, 5 links, 4 joints
Joints:
- joint base_to_deltat: origin xyz=0 0 -0.65 rpy=3.14159 0 0 -> xyz=0 0 -0.65 rpy=3.14159 0 3.14159
